Commit message: update

File: urdf/lux.urdf (robot description, URDF)
Before this commit: robot 4_legged_robot, 13 links, 12 joints
Links:
- link 1_link1: geometry visual mesh filename=package://lux_description/meshes/link1.dae scale=1 1 1
- link 1_link2: geometry visual mesh filename=package://lux_description/meshes/link2.dae scale=1 1 1
- link 1_link3: geometry visual mesh filename=package://lux_description/meshes/link3.dae scale=1 1 1
- link 2_link1: mass None -> 0; geometry visual mesh filename=package://lux_description/meshes/link1.dae scale=1 1 1
- link 2_link2: geometry visual mesh filename=package://lux_description/meshes/link2.dae scale=1 1 1
- link 2_link3: geometry visual mesh filename=package://lux_description/meshes/link3.dae scale=1 1 1
- link 3_link1: mass None -> 0; geometry visual mesh filename=package://lux_description/meshes/link1.dae scale=1 1 1
- link 3_link2: geometry visual mesh filename=package://lux_description/meshes/link2.dae scale=1 1 1
- link 3_link3: geometry visual mesh filename=package://lux_description/meshes/link3.dae scale=1 1 1
- link 4_link1: mass None -> 0; geometry visual mesh filename=package://lux_description/meshes/link1.dae scale=1 1 1
- link 4_link2: mass None -> 0; geometry visual mesh filename=package://lux_description/meshes/link2.dae scale=1 1 1
- link 4_link3: geometry visual mesh filename=package://lux_description/meshes/link3.dae scale=1 1 1
- link base_link: mass 0 -> None; geometry visual mesh filename=package://lux_description/meshes/body.dae scale=1 1 1

Commit message: feat: update

File: urdf/lux.urdf (robot description, URDF)
Before this commit: robot 4_legged_robot, 13 links, 12 joints
Links:
- added link world
- link 1_link1: geometry collision mesh filename=package://lux_description/meshes/link1.dae scale=1 1 1; visual mesh filename=package://lux_description/meshes/link1.dae scale=1 1 1
- link 1_link2: geometry collision mesh filename=package://lux_description/meshes/link2.dae scale=1 1 1; visual mesh filename=package://lux_description/meshes/link2.dae scale=1 1 1
- link 1_link3: geometry collision mesh filename=package://lux_description/meshes/link3.dae scale=1 1 1; visual mesh filename=package://lux_description/meshes/link3.dae scale=1 1 1
- link 2_link1: geometry collision mesh filename=package://lux_description/meshes/link1.dae scale=1 1 1; visual mesh filename=package://lux_description/meshes/link1.dae scale=1 1 1
- link 2_link3: geometry collision mesh filename=package://lux_description/meshes/link3.dae scale=1 1 1; visual mesh filename=package://lux_description/meshes/link3.dae scale=1 1 1
- link 3_link1: geometry collision mesh filename=package://lux_description/meshes/link1.dae scale=1 1 1; visual mesh filename=package://lux_description/meshes/link1.dae scale=1 1 1
- link 3_link3: geometry collision mesh filename=package://lux_description/meshes/link3.dae scale=1 1 1; visual mesh filename=package://lux_description/meshes/link3.dae scale=1 1 1
- link 4_link1: geometry collision mesh filename=package://lux_description/meshes/link1.dae scale=1 1 1; visual mesh filename=package://lux_description/meshes/link1.dae scale=1 1 1
- link 4_link3: geometry collision mesh filename=package://lux_description/meshes/link3.dae scale=1 1 1; visual mesh filename=package://lux_description/meshes/link3.dae scale=1 1 1
- link base_link: mass None -> 1; geometry collision mesh filename=package://lux_description/meshes/body.dae scale=1 1 1; visual mesh filename=package://lux_description/meshes/body.dae scale=1 1 1
Joints:
- added joint world_joint: type fixed, parent world, child base_link, origin xyz=0 0 0 rpy=0 0 0
